File: Hardware/LilyPad_Arduino_SimpleSnap.brd (EAGLE design)
At the start: 50 x 50 mm, 45 parts, among them U1 ATMEGA328, U2 MCP73831, Y1 8MHz

Commit message: Fixing resistor value to match actual BOM
Parts:
- R2: value 1k -> 10k
Changed lines of the file:
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@@
 <?xml version="1.0" encoding="utf-8"?>
 <!DOCTYPE eagle SYSTEM "eagle.dtd">
-<eagle version="7.2.0">
+<eagle version="7.6.0">
 <drawing>
 <settings>
@@
 <element name="PP-SCK" library="SparkFun" package="PAD.03X.05" value="" x="-8.526" y="-2" rot="MR180"/>
 <element name="PP-RST" library="SparkFun" package="PAD.03X.05" value="" x="9.32" y="-11.32" rot="MR0"/>
-<element name="R2" library="SparkFun" package="0402-RES" value="1k" x="-12.46" y="-7" rot="MR90"/>
+<element name="R2" library="SparkFun" package="0402-RES" value="10k" x="-12.46" y="-7" rot="MR90"/>
 <element name="TP-FTDI_VCC" library="SparkFun" package="PAD.03X.05" value="" x="-1.3" y="10.77" rot="MR0"/>
 <element name="JP3" library="SparkFun" package="SNAP-FEMALE" value="M01SNAP-FEMALE_LARGE" x="18.8303" y="8.5995" rot="MR0"/>
