File: Hardware/LilyPad_Arduino_SimpleSnap.sch (EAGLE design)
At the start: 45 parts, among them U1 ATMEGA328, U2 MCP73831, Y1 8MHz

Commit message: Fixing resistor value to match actual BOM
Parts:
- R2: value 1k -> 10k
Changed lines of the file:
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@@
 <?xml version="1.0" encoding="utf-8"?>
 <!DOCTYPE eagle SYSTEM "eagle.dtd">
-<eagle version="7.2.0">
+<eagle version="7.6.0">
 <drawing>
 <settings>
@@
 <part name="PP-RST" library="SparkFun" deviceset="TEST-POINT" device="3X5" value=""/>
 <part name="GND1" library="supply1" deviceset="GND" device=""/>
-<part name="R2" library="SparkFun" deviceset="RESISTOR" device="0402-RES" value="1k"/>
+<part name="R2" library="SparkFun" deviceset="RESISTOR" device="0402-RES" value="10k"/>
 <part name="GND13" library="supply1" deviceset="GND" device=""/>
 <part name="TP-FTDI_VCC" library="SparkFun" deviceset="TEST-POINT" device="3X5" value=""/>
